File: hardware/cm1/cm1.brd (EAGLE design)
At the start: 35.2 x 48.2 mm, 18 parts, among them Q2 BC338, Q3 BC338

Commit message: removed pull up transistor from cm1
Parts:
- removed D1: (no value), SparkFun-DiscreteSemi:DIODE-1N4148
- removed Q2: BC338, transistor-npn:TO92-EBC
- removed R3: 10R, SparkFun-Passives:AXIAL-0.4
- R1, R2: value 2k2 -> 1k5
- SJ1: value SOLDERJUMPERTRACE-PTH -> SOLDERJUMPERPTH; device SparkFun-Passives:SJ_2S-TRACE-PTH -> SparkFun-Passives:SJ_2S-PTH
- moved R2 4.58 mm to (25.4, 22.9), turned to 180 degrees
Connections:
- removed net N$6: IRF4905.G, R3.P$2
- removed net N$8: D1.A, Q2.E, R3.P$1
- net N$10: now also R2.P$2; no longer Q2.C, R2.P$1
- net N$9: now also IRF4905.G, R2.P$1; no longer D1.C, Q2.B, R2.P$2
Routing:
- net N$6: track 17.3 -> 0.00 mm
- net N$8: track 16.3 -> 0.00 mm
- net N$4: track 21.2 -> 9.03 mm
- net N$10: track 51.2 -> 39.7 mm
- net N$9: track 21.9 -> 19.4 mm
Other:
- board text added: "+12V"
- board text added: "CTRL"
- board text added: "OUT"

Commit message: fixed wrong transistor
Parts:
- Q3: value BC338 -> 2N3904; device transistor-npn:TO92-EBC -> transistor:TO92
- moved Q3 2.54 mm to (29.2, 36.8), turned to 270 degrees
Connections:
- net GND: now also Q3.3; no longer Q3.E
- net N$5: now also Q3.2; no longer Q3.B
- net N$9: now also Q3.1; no longer Q3.C
Routing:
- net N$5: track 14.3 -> 16.7 mm
- net N$9: track 19.4 -> 20.1 mm
Changed lines of the file:
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@@
 <element name="STANDOFF2" library="SparkFun-Electromechanical" package="STAND-OFF" value="STAND-OFF" x="3.81" y="3.81"/>
 <element name="SJ1" library="SparkFun-Passives" package="SJ_2S-PTH" value="SOLDERJUMPERPTH" x="11.43" y="29.21" smashed="yes" rot="R270"/>
-<element name="Q3" library="transistor-npn" package="TO92-EBC" value="BC338" x="26.67" y="36.83" rot="R90"/>
+<element name="Q3" library="transistor" package="TO92" value="2N3904" x="29.21" y="36.83" rot="R270"/>
 <element name="R1" library="SparkFun-Passives" package="AXIAL-0.4" value="1k5" x="21.59" y="31.75" smashed="yes" rot="R90">
 <attribute name="NAME" x="24.765" y="28.575" size="0.8128" layer="25" font="vector" ratio="15" rot="R90"/>
@@
 <contactref element="12_IN" pad="1"/>
 <contactref element="12V_OUT" pad="2"/>
-<contactref element="Q3" pad="E"/>
+<contactref element="Q3" pad="3"/>
 <contactref element="CTRL" pad="1"/>
 <contactref element="C2" pad="2"/>
@@
 </signal>
 <signal name="N$9">
-<contactref element="Q3" pad="C"/>
+<contactref element="Q3" pad="1"/>
 <contactref element="R2" pad="P$1"/>
 <contactref element="IRF4905" pad="G"/>
-<wire x1="27.94" y1="34.29" x2="27.94" y2="25.4" width="1.4224" layer="1"/>
-<wire x1="27.94" y1="25.4" x2="30.48" y2="22.86" width="1.4224" layer="1"/>
 <wire x1="30.48" y1="22.86" x2="30.48" y2="17.78" width="1.4224" layer="1"/>
 <wire x1="30.48" y1="17.78" x2="31.75" y2="16.51" width="1.4224" layer="1"/>
+<wire x1="30.48" y1="22.86" x2="30.48" y2="34.29" width="1.27" layer="1"/>
+<wire x1="30.48" y1="34.29" x2="29.21" y2="35.56" width="1.27" layer="1"/>
 </signal>
 <signal name="N$10">
@@
 <signal name="N$5">
 <contactref element="R1" pad="P$1"/>
-<contactref element="Q3" pad="B"/>
-<wire x1="21.59" y1="26.67" x2="21.59" y2="33.02" width="1.27" layer="1"/>
-<wire x1="21.59" y1="33.02" x2="25.4" y2="36.83" width="1.27" layer="1"/>
-<wire x1="25.4" y1="36.83" x2="27.94" y2="36.83" width="1.27" layer="1"/>
+<contactref element="Q3" pad="2"/>
+<wire x1="31.115" y1="36.83" x2="26.67" y2="36.83" width="0.8128" layer="1"/>
+<wire x1="26.67" y1="36.83" x2="25.4" y2="35.56" width="0.8128" layer="1"/>
+<wire x1="25.4" y1="35.56" x2="25.4" y2="30.48" width="0.8128" layer="1"/>
+<wire x1="25.4" y1="30.48" x2="21.59" y2="26.67" width="0.8128" layer="1"/>
 </signal>
 <signal name="N$6">
