File: hardware/cm1/cm1.sch (EAGLE design)
At the start: 18 parts, among them Q2 BC338, Q3 BC338

Commit message: removed pull up transistor from cm1
Parts:
- removed D1: (no value), SparkFun-DiscreteSemi:DIODE1N4148
- removed Q2: BC338, transistor-npn:BC338
- removed R3: 10R, SparkFun-Passives:RESISTORPTH-1/4W
- R1, R2: value 2k2 -> 1k5
- SJ1: value SOLDERJUMPERTRACE-PTH -> SOLDERJUMPERPTH; device SparkFun-Passives:SOLDERJUMPERTRACE-PTH -> SparkFun-Passives:SOLDERJUMPERPTH
Connections:
- removed net N$6: IRF4905.G, R3.2
- removed net N$8: D1.A, Q2.E, R3.1
- net N$10: now also R2.2; no longer Q2.C, R2.1
- net N$9: now also IRF4905.G, R2.1; no longer D1.C, Q2.B, R2.2
Other:
- moved on the sheet: D2, R2
Changed lines of the file:
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@@
 <part name="STANDOFF1" library="SparkFun-Electromechanical" deviceset="STAND-OFF" device=""/>
 <part name="STANDOFF2" library="SparkFun-Electromechanical" deviceset="STAND-OFF" device=""/>
-<part name="SJ1" library="SparkFun-Passives" deviceset="SOLDERJUMPER" device="TRACE-PTH"/>
-<part name="Q2" library="transistor-npn" deviceset="BC338*" device=""/>
+<part name="SJ1" library="SparkFun-Passives" deviceset="SOLDERJUMPER" device="PTH" value="SOLDERJUMPERPTH"/>
 <part name="Q3" library="transistor-npn" deviceset="BC338*" device=""/>
-<part name="D1" library="SparkFun-DiscreteSemi" deviceset="DIODE" device="1N4148"/>
-<part name="R1" library="SparkFun-Passives" deviceset="RESISTOR" device="PTH-1/4W" value="2k2"/>
-<part name="R2" library="SparkFun-Passives" deviceset="RESISTOR" device="PTH-1/4W" value="2k2"/>
-<part name="R3" library="SparkFun-Passives" deviceset="RESISTOR" device="PTH-1/4W" value="10R"/>
+<part name="R1" library="SparkFun-Passives" deviceset="RESISTOR" device="PTH-1/4W" value="1k5"/>
 <part name="IRF4905" library="transistor-power" deviceset="PMOSFET_P" device="TO220BV"/>
 <part name="D2" library="diode" deviceset="1N581*" device="" technology="9-B"/>
 <part name="C2" library="SparkFun-Capacitors" deviceset="CAP" device="PTH" value="3.3u/100V"/>
 <part name="C1" library="PowerBoard" deviceset="CPOL" device="7343"/>
+<part name="R2" library="SparkFun-Passives" deviceset="RESISTOR" device="PTH-1/4W" value="1k5"/>
 </parts>
 <sheets>
@@
 <attribute name="NAME" x="38.1" y="83.82" size="1.778" layer="95"/>
 </instance>
-<instance part="Q2" gate="G$1" x="55.88" y="40.64"/>
 <instance part="Q3" gate="G$1" x="43.18" y="25.4"/>
-<instance part="D1" gate="G$1" x="50.8" y="35.56" rot="R180"/>
 <instance part="R1" gate="G$1" x="30.48" y="25.4" rot="R180"/>
-<instance part="R2" gate="G$1" x="45.72" y="45.72" rot="R270"/>
-<instance part="R3" gate="G$1" x="63.5" y="35.56"/>
-<instance part="IRF4905" gate="G$1" x="73.66" y="38.1"/>
-<instance part="D2" gate="G$1" x="81.28" y="38.1" rot="R90"/>
+<instance part="IRF4905" gate="G$1" x="73.66" y="38.1" smashed="yes">
+<attribute name="NAME" x="63.5" y="43.18" size="1.778" layer="95"/>
+<attribute name="VALUE" x="78.74" y="38.1" size="1.778" layer="96"/>
+</instance>
+<instance part="D2" gate="G$1" x="81.28" y="40.64" smashed="yes" rot="R90">
+<attribute name="NAME" x="86.995" y="38.354" size="1.778" layer="95" rot="R90"/>
+<attribute name="VALUE" x="96.266" y="46.609" size="1.778" layer="96" rot="R180"/>
+</instance>
 <instance part="C2" gate="G$1" x="30.48" y="63.5"/>
 <instance part="C1" gate="G$1" x="66.04" y="63.5"/>
+<instance part="R2" gate="G$1" x="60.96" y="50.8"/>
 </instances>
 <busses>
@@
 <junction x="76.2" y="33.02"/>
 <pinref part="D2" gate="G$1" pin="A"/>
-<wire x1="81.28" y1="35.56" x2="81.28" y2="33.02" width="0.1524" layer="91"/>
+<wire x1="81.28" y1="38.1" x2="81.28" y2="33.02" width="0.1524" layer="91"/>
 <wire x1="81.28" y1="33.02" x2="76.2" y2="33.02" width="0.1524" layer="91"/>
-</segment>
-</net>
-<net name="N$8" class="0">
-<segment>
-<pinref part="R3" gate="G$1" pin="1"/>
-<pinref part="Q2" gate="G$1" pin="E"/>
-<pinref part="D1" gate="G$1" pin="A"/>
-<wire x1="53.34" y1="35.56" x2="58.42" y2="35.56" width="0.1524" layer="91"/>
-<junction x="58.42" y="35.56"/>
 </segment>
 </net>
 <net name="N$9" class="0">
 <segment>
-<pinref part="R2" gate="G$1" pin="2"/>
 <pinref part="Q3" gate="G$1" pin="C"/>
-<wire x1="45.72" y1="40.64" x2="45.72" y2="35.56" width="0.1524" layer="91"/>
-<pinref part="D1" gate="G$1" pin="C"/>
-<wire x1="45.72" y1="35.56" x2="45.72" y2="30.48" width="0.1524" layer="91"/>
-<wire x1="48.26" y1="35.56" x2="45.72" y2="35.56" width="0.1524" layer="91"/>
-<junction x="45.72" y="35.56"/>
-<pinref part="Q2" gate="G$1" pin="B"/>
-<wire x1="53.34" y1="40.64" x2="45.72" y2="40.64" width="0.1524" layer="91"/>
+<wire x1="45.72" y1="30.48" x2="45.72" y2="40.64" width="0.1524" layer="91"/>
+<pinref part="R2" gate="G$1" pin="1"/>
+<wire x1="45.72" y1="40.64" x2="45.72" y2="50.8" width="0.1524" layer="91"/>
+<wire x1="45.72" y1="50.8" x2="55.88" y2="50.8" width="0.1524" layer="91"/>
+<pinref part="IRF4905" gate="G$1" pin="G"/>
+<wire x1="68.58" y1="40.64" x2="45.72" y2="40.64" width="0.1524" layer="91"/>
 <junction x="45.72" y="40.64"/>
 </segment>
@@
 <net name="N$10" class="0">
 <segment>
-<pinref part="R2" gate="G$1" pin="1"/>
-<pinref part="Q2" gate="G$1" pin="C"/>
-<wire x1="45.72" y1="50.8" x2="58.42" y2="50.8" width="0.1524" layer="91"/>
-<wire x1="58.42" y1="50.8" x2="58.42" y2="45.72" width="0.1524" layer="91"/>
 <pinref part="LM2940-12" gate="G$1" pin="OUT"/>
 <wire x1="48.26" y1="71.12" x2="66.04" y2="71.12" width="0.1524" layer="91"/>
@@
 <wire x1="45.72" y1="81.28" x2="66.04" y2="81.28" width="0.1524" layer="91"/>
 <wire x1="66.04" y1="81.28" x2="66.04" y2="71.12" width="0.1524" layer="91"/>
-<wire x1="76.2" y1="43.18" x2="76.2" y2="50.8" width="0.1524" layer="91"/>
 <wire x1="76.2" y1="50.8" x2="76.2" y2="71.12" width="0.1524" layer="91"/>
 <wire x1="76.2" y1="71.12" x2="66.04" y2="71.12" width="0.1524" layer="91"/>
-<wire x1="58.42" y1="50.8" x2="76.2" y2="50.8" width="0.1524" layer="91"/>
-<junction x="58.42" y="50.8"/>
-<junction x="76.2" y="50.8"/>
-<pinref part="IRF4905" gate="G$1" pin="S"/>
-<junction x="76.2" y="43.18"/>
 <pinref part="D2" gate="G$1" pin="C"/>
-<wire x1="81.28" y1="40.64" x2="81.28" y2="50.8" width="0.1524" layer="91"/>
+<wire x1="81.28" y1="43.18" x2="81.28" y2="50.8" width="0.1524" layer="91"/>
 <wire x1="81.28" y1="50.8" x2="76.2" y2="50.8" width="0.1524" layer="91"/>
 <pinref part="C1" gate="G$1" pin="+"/>
+<pinref part="IRF4905" gate="G$1" pin="S"/>
+<wire x1="76.2" y1="43.18" x2="76.2" y2="50.8" width="0.1524" layer="91"/>
+<junction x="76.2" y="50.8"/>
+<pinref part="R2" gate="G$1" pin="2"/>
+<wire x1="66.04" y1="50.8" x2="76.2" y2="50.8" width="0.1524" layer="91"/>
 </segment>
 </net>
@@
 </segment>
 </net>
-<net name="N$6" class="0">
-<segment>
-<pinref part="IRF4905" gate="G$1" pin="G"/>
-<pinref part="R3" gate="G$1" pin="2"/>
-<wire x1="68.58" y1="40.64" x2="68.58" y2="35.56" width="0.1524" layer="91"/>
-</segment>
-</net>

Commit message: fixed wrong transistor
Parts:
- Q3: value BC338 -> 2N3904; device transistor-npn:BC338 -> transistor:2N3904
Changed lines of the file:
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@@
 <part name="STANDOFF2" library="SparkFun-Electromechanical" deviceset="STAND-OFF" device=""/>
 <part name="SJ1" library="SparkFun-Passives" deviceset="SOLDERJUMPER" device="PTH" value="SOLDERJUMPERPTH"/>
-<part name="Q3" library="transistor-npn" deviceset="BC338*" device=""/>
+<part name="Q3" library="transistor" deviceset="2N3904" device=""/>
 <part name="R1" library="SparkFun-Passives" deviceset="RESISTOR" device="PTH-1/4W" value="1k5"/>
 <part name="IRF4905" library="transistor-power" deviceset="PMOSFET_P" device="TO220BV"/>
@@
 <attribute name="NAME" x="38.1" y="83.82" size="1.778" layer="95"/>
 </instance>
-<instance part="Q3" gate="G$1" x="43.18" y="25.4"/>
+<instance part="Q3" gate="G1" x="43.18" y="25.4"/>
 <instance part="R1" gate="G$1" x="30.48" y="25.4" rot="R180"/>
 <instance part="IRF4905" gate="G$1" x="73.66" y="38.1" smashed="yes">
@@
 </segment>
 <segment>
-<pinref part="Q3" gate="G$1" pin="E"/>
+<pinref part="Q3" gate="G1" pin="E"/>
 <pinref part="GND5" gate="1" pin="GND"/>
 <wire x1="45.72" y1="20.32" x2="45.72" y2="17.78" width="0.1524" layer="91"/>
@@
 <net name="N$9" class="0">
 <segment>
-<pinref part="Q3" gate="G$1" pin="C"/>
+<pinref part="Q3" gate="G1" pin="C"/>
 <wire x1="45.72" y1="30.48" x2="45.72" y2="40.64" width="0.1524" layer="91"/>
 <pinref part="R2" gate="G$1" pin="1"/>
@@
 <segment>
 <pinref part="R1" gate="G$1" pin="1"/>
-<pinref part="Q3" gate="G$1" pin="B"/>
+<pinref part="Q3" gate="G1" pin="B"/>
 <wire x1="35.56" y1="25.4" x2="40.64" y2="25.4" width="0.1524" layer="91"/>
 </segment>
